Commit message: Added collision meshes to the base

File: eve_r3_description/urdf.in/eve_r3_leg.in.urdf (robot description, URDF)
Before this commit: robot eve_r3_leg, 9 links, 8 joints
Links:
- link base: geometry collision sphere radius=0.1524; visual mesh filename=package://eve_r3_description/meshes/base.obj scale=1 1 1
- link l_wheel: geometry collision cylinder length=0.03 radius=0.1524; visual mesh filename=package://eve_r3_description/meshes/wheel.obj scale=1 1 1
- link r_wheel: geometry collision cylinder length=0.03 radius=0.1524; visual mesh filename=package://eve_r3_description/meshes/wheel.obj scale=1 1 1

File: eve_r3_description/urdf/eve_r3.urdf (robot description, URDF)
Before this commit: robot eve_r3, 96 links, 95 joints
Links:
- link base: geometry collision sphere radius=0.1524; visual mesh filename=package://eve_r3_description/meshes/base.obj scale=1 1 1
- link l_wheel: geometry collision cylinder length=0.03 radius=0.1524; visual mesh filename=package://eve_r3_description/meshes/wheel.obj scale=1 1 1
- link r_wheel: geometry collision cylinder length=0.03 radius=0.1524; visual mesh filename=package://eve_r3_description/meshes/wheel.obj scale=1 1 1
