Commit message: Generated SDF and URDF models from templates

File: eve_r3_description/urdf.in/eve_r3_upper_body.in.urdf (robot description, URDF)
Before this commit: robot eve_r3_upper_body, 1 links, 0 joints
Links:
- link pelvis: mass 10.04177517 -> 10.12075049

File: eve_r3_description/urdf/eve_r3.urdf (robot description, URDF)
Before this commit: robot eve_r3, 96 links, 95 joints
Links:
- link abdomen: mass 3.4381772 -> 3.429553
- link ankle_y_link: mass 2.656189 -> 2.742145
- link base: mass 13.647499 -> 12.487535
- link head: mass 2.355 -> 1.84975554
- link hip_x_link: mass 2.868669 -> 2.94819561
- link l_elbow: mass 0.46261553 -> 0.46228452
- link l_lower_arm: mass 1.63933464 -> 1.72646966
- link l_palm: mass 0.1486378 -> 0.22529206
- link l_scapula: mass 2.75566786 -> 3.00902868
- link l_shoulder: mass 0.70265653 -> 0.62091759
- link l_upper_arm: mass 2.92531724 -> 3.32260186
- link l_wheel: mass 1.52693 -> 2.17850874
- link l_wrist: mass 0.30363399 -> 0.3582051
- link pelvis: mass 10.11628645 -> 10.12075049
- link r_elbow: mass 0.46261553 -> 0.4622891
- link r_lower_arm: mass 1.63933464 -> 1.72645167
- link r_palm: mass 0.1486378 -> 0.22529206
- link r_scapula: mass 2.75566786 -> 3.00220101
- link r_shoulder: mass 0.70264272 -> 0.62091759
- link r_upper_arm: mass 2.92531724 -> 3.32084455
- link r_wheel: mass 1.52693 -> 2.17850874
- link r_wrist: mass 0.30363399 -> 0.3582051
- link shin: mass 10.894892 -> 11.06513851
- link thigh: mass 12.846698 -> 10.80882706
Joints:
- joint j_l_elbow_y: origin xyz=0.0 0.0 -0.313989 rpy=0.0 0.0 0.0 -> xyz=0.0 0.0 -0.3141 rpy=0.0 0.0 0.0
- joint j_l_shoulder_x: origin xyz=0.0 0.0 0.0 rpy=-0.253261563 0.0 0.0 -> xyz=0.0 0.0 0.0 rpy=-0.261799 0.0 0.0
- joint j_l_shoulder_y: origin xyz=0.010525 0.207221 0.545525 rpy=0.253261563 0.0 -0.261799 -> xyz=0.01041 0.20675 0.54735 rpy=0.261799 0.0 -0.261799
- joint j_neck_y: axis 0.0 1 0.0 -> 0.0 1.0 0.0; origin xyz=-0.004458 0.0 0.680766 rpy=0.0 0.0 0.0 -> xyz=0.00646 0.00085 0.67201 rpy=0.0 0.0 0.0
- joint j_r_elbow_y: axis 0.0 1 0.0 -> 0.0 1.0 0.0; origin xyz=0.0 0.0 -0.313989 rpy=0.0 0.0 0.0 -> xyz=0.0 0.0 -0.3141 rpy=0.0 0.0 0.0
- joint j_r_elbow_z: axis 0.0 0.0 1 -> 0.0 0.0 1.0
- joint j_r_shoulder_x: origin xyz=0.0 0.0 0.0 rpy=0.253261563 0.0 0.0 -> xyz=0.0 0.0 0.0 rpy=0.261799 0.0 0.0
- joint j_r_shoulder_y: origin xyz=0.010525 -0.207221 0.545525 rpy=-0.253261563 0.0 0.261799 -> xyz=0.01041 -0.20675 0.54735 rpy=-0.261799 0.0 0.261799
- joint j_r_wrist_x: axis 1 0.0 0.0 -> 1.0 0.0 0.0
- joint j_r_wrist_y: axis 0.0 1 0.0 -> 0.0 1.0 0.0; origin xyz=0.0 0.0 -0.292850 rpy=0.0 0.0 0.0 -> xyz=0.0 0.0 -0.29285 rpy=0.0 0.0 0.0

File: eve_r3_description/urdf/eve_r3_upper_body.urdf (robot description, URDF)
Before this commit: robot eve_r3_upper_body, 87 links, 86 joints
Links:
- link l_elbow: mass 0.46261553 -> 0.46228452
- link l_lower_arm: mass 1.63933464 -> 1.72646966
- link l_palm: mass 0.1486378 -> 0.22529206
- link l_scapula: mass 2.75566786 -> 3.00902868
- link l_shoulder: mass 0.70265653 -> 0.62091759
- link l_upper_arm: mass 2.92531724 -> 3.32260186
- link l_wrist: mass 0.30363399 -> 0.3582051
- link pelvis: mass 10.04177517 -> 10.12075049
- link r_elbow: mass 0.46261553 -> 0.4622891
- link r_lower_arm: mass 1.63933464 -> 1.72645167
- link r_palm: mass 0.1486378 -> 0.22529206
- link r_scapula: mass 2.75566786 -> 3.00220101
- link r_shoulder: mass 0.70264272 -> 0.62091759
- link r_upper_arm: mass 2.92531724 -> 3.32084455
- link r_wrist: mass 0.30363399 -> 0.3582051
Joints:
- joint j_l_elbow_y: origin xyz=0.0 0.0 -0.313989 rpy=0.0 0.0 0.0 -> xyz=0.0 0.0 -0.3141 rpy=0.0 0.0 0.0
- joint j_l_shoulder_x: origin xyz=0.0 0.0 0.0 rpy=-0.253261563 0.0 0.0 -> xyz=0.0 0.0 0.0 rpy=-0.261799 0.0 0.0
- joint j_l_shoulder_y: origin xyz=0.010525 0.207221 0.545525 rpy=0.253261563 0.0 -0.261799 -> xyz=0.01041 0.20675 0.54735 rpy=0.261799 0.0 -0.261799
- joint j_r_elbow_y: axis 0.0 1 0.0 -> 0.0 1.0 0.0; origin xyz=0.0 0.0 -0.313989 rpy=0.0 0.0 0.0 -> xyz=0.0 0.0 -0.3141 rpy=0.0 0.0 0.0
- joint j_r_elbow_z: axis 0.0 0.0 1 -> 0.0 0.0 1.0
- joint j_r_shoulder_x: origin xyz=0.0 0.0 0.0 rpy=0.253261563 0.0 0.0 -> xyz=0.0 0.0 0.0 rpy=0.261799 0.0 0.0
- joint j_r_shoulder_y: origin xyz=0.010525 -0.207221 0.545525 rpy=-0.253261563 0.0 0.261799 -> xyz=0.01041 -0.20675 0.54735 rpy=-0.261799 0.0 0.261799
- joint j_r_wrist_x: axis 1 0.0 0.0 -> 1.0 0.0 0.0
- joint j_r_wrist_y: axis 0.0 1 0.0 -> 0.0 1.0 0.0; origin xyz=0.0 0.0 -0.292850 rpy=0.0 0.0 0.0 -> xyz=0.0 0.0 -0.29285 rpy=0.0 0.0 0.0

Commit message: Updated upper body to include head and yaw joint

File: eve_r3_description/urdf.in/eve_r3_upper_body.in.urdf (robot description, URDF)
Before this commit: robot eve_r3_upper_body, 1 links, 0 joints
Links:
- added link abdomen, mass 3.4381772; visual mesh filename=package://eve_r3_description/meshes/abdomen.obj scale=1 1 1
Joints:
- added joint j_hip_z: type revolute, parent abdomen, child pelvis, origin xyz=0.0 0.0 0.0 rpy=0.0 0.0 0.0, axis 0.0 0.0 1.0, limit lower=-1.0472 upper=1.0472 effort=-1.0 velocity=-1.0

File: eve_r3_description/urdf/eve_r3_upper_body.urdf (robot description, URDF)
Before this commit: robot eve_r3_upper_body, 87 links, 86 joints
Links:
- added link abdomen, mass 3.4381772; visual mesh filename=package://eve_r3_description/meshes/abdomen.obj scale=1 1 1
- added link head, mass 2.355; visual mesh filename=package://eve_r3_description/meshes/head.obj scale=1 1 1
Joints:
- added joint j_hip_z: type revolute, parent abdomen, child pelvis, origin xyz=0.0 0.0 0.0 rpy=0.0 0.0 0.0, axis 0.0 0.0 1.0, limit lower=-1.0472 upper=1.0472 effort=-1.0 velocity=-1.0
- added joint j_neck_y: type revolute, parent pelvis, child head, origin xyz=-0.004458 0.0 0.680766 rpy=0.0 0.0 0.0, axis 0.0 1 0.0, limit lower=-0.0872664626 upper=0.698132 effort=-1.0 velocity=-1.0

Commit message: Updated upper body to include head and yaw joint
# Conflicts:
#	build.gradle
#	eve_r3_description/urdf.in/eve_r3_upper_body.in.urdf

File: eve_r3_description/urdf.in/eve_r3_upper_body.in.urdf (robot description, URDF)
Before this commit: robot eve_r3_upper_body, 1 links, 0 joints
Links:
- added link abdomen, mass 3.429553; visual mesh filename=package://eve_r3_description/meshes/abdomen.obj scale=1 1 1
Joints:
- added joint j_hip_z: type revolute, parent abdomen, child pelvis, origin xyz=0.0 0.0 0.0 rpy=0.0 0.0 0.0, axis 0.0 0.0 1.0, limit lower=-1.0472 upper=1.0472 effort=-1.0 velocity=-1.0

File: eve_r3_description/urdf/eve_r3_upper_body.urdf (robot description, URDF)
Before this commit: robot eve_r3_upper_body, 87 links, 86 joints
Links:
- added link abdomen, mass 3.429553; visual mesh filename=package://eve_r3_description/meshes/abdomen.obj scale=1 1 1
- added link head, mass 1.84975554; visual mesh filename=package://eve_r3_description/meshes/head.obj scale=1 1 1
Joints:
- added joint j_hip_z: type revolute, parent abdomen, child pelvis, origin xyz=0.0 0.0 0.0 rpy=0.0 0.0 0.0, axis 0.0 0.0 1.0, limit lower=-1.0472 upper=1.0472 effort=-1.0 velocity=-1.0
- added joint j_neck_y: type revolute, parent pelvis, child head, origin xyz=0.00646 0.00085 0.67201 rpy=0.0 0.0 0.0, axis 0.0 1.0 0.0, limit lower=-0.0872664626 upper=0.698132 effort=-1.0 velocity=-1.0
