Commit message: Henrique's update March 2020
Updated inertia values for each subassembly. Current values do not include inertia/masses of cosmetic covers

File: eve_r3_description/urdf.in/eve_r3_head.in.urdf (robot description, URDF)
Before this commit: robot eve_r3_head, 1 links, 1 joints
Links:
- added link Root_1, mass 0.0; visual mesh filename=package:// scale=1 1 1
- link head: mass 2.355 -> 1.45569784
Joints:
- joint j_neck_y: axis 0.0 1 0.0 -> 0.0 1.0 0.0; parent pelvis -> Root_1

File: eve_r3_description/urdf.in/eve_r3_left_arm.in.urdf (robot description, URDF)
Before this commit: robot eve_r3_left_arm, 7 links, 7 joints
Links:
- link l_elbow: mass 0.46261553 -> 0.46228452
- link l_lower_arm: mass 1.63933464 -> 1.72646966
- link l_palm: mass 0.1486378 -> 0.22529206
- link l_scapula: mass 2.75566786 -> 3.00902868
- link l_shoulder: mass 0.70265653 -> 0.62091759
- link l_upper_arm: mass 2.92531724 -> 3.32260186
- link l_wrist: mass 0.30363399 -> 0.3582051
Joints:
- joint j_l_shoulder_y: parent pelvis -> l_shoulder

File: eve_r3_description/urdf.in/eve_r3_leg.in.urdf (robot description, URDF)
Before this commit: robot eve_r3_leg, 9 links, 8 joints
Links:
- link abdomen: mass 3.4381772 -> 3.429553
- link ankle_y_link: mass 2.656189 -> 2.742145
- link base: mass 13.647499 -> 12.487535
- link hip_x_link: mass 2.868669 -> 2.94819561
- link l_wheel: mass 1.52693 -> 2.17850874
- link pelvis: mass 10.11628645 -> 10.12075049
- link r_wheel: mass 1.52693 -> 2.17850874
- link shin: mass 10.894892 -> 11.06513851
- link thigh: mass 12.846698 -> 10.80882706

File: eve_r3_description/urdf.in/eve_r3_right_arm.in.urdf (robot description, URDF)
Before this commit: robot eve_r3_right_arm, 7 links, 7 joints
Links:
- link r_elbow: mass 0.46261553 -> 0.4622891
- link r_lower_arm: mass 1.63933464 -> 1.72645167
- link r_palm: mass 0.1486378 -> 0.22529206
- link r_scapula: mass 2.75566786 -> 3.00220101
- link r_shoulder: mass 0.70264272 -> 0.62091759
- link r_upper_arm: mass 2.92531724 -> 3.32084455
- link r_wrist: mass 0.30363399 -> 0.3582051
Joints:
- joint j_r_elbow_y: axis 0.0 1 0.0 -> 0.0 1.0 0.0
- joint j_r_elbow_z: axis 0.0 0.0 1 -> 0.0 0.0 1.0
- joint j_r_shoulder_y: parent pelvis -> r_shoulder
- joint j_r_wrist_x: axis 1 0.0 0.0 -> 1.0 0.0 0.0
- joint j_r_wrist_y: axis 0.0 1 0.0 -> 0.0 1.0 0.0; origin xyz=0.0 0.0 -0.292850 rpy=0.0 0.0 0.0 -> xyz=0.0 0.0 -0.29285 rpy=0.0 0.0 0.0

Commit message: Fixed origin joint

File: eve_r3_description/urdf.in/eve_r3_head.in.urdf (robot description, URDF)
Before this commit: robot eve_r3_head, 2 links, 1 joints
Links:
- removed link Root_1
Joints:
- joint j_neck_y: parent Root_1 -> pelvis

File: eve_r3_description/urdf.in/eve_r3_left_arm.in.urdf (robot description, URDF)
Before this commit: robot eve_r3_left_arm, 7 links, 7 joints
Joints:
- joint j_l_shoulder_y: parent l_shoulder -> pelvis

File: eve_r3_description/urdf.in/eve_r3_right_arm.in.urdf (robot description, URDF)
Before this commit: robot eve_r3_right_arm, 7 links, 7 joints
Joints:
- joint j_r_shoulder_y: parent r_shoulder -> pelvis

Commit message: updated arm and head offsets

File: eve_r3_description/urdf.in/eve_r3_head.in.urdf (robot description, URDF)
Before this commit: robot eve_r3_head, 1 links, 1 joints
Links:
- link head: mass 1.45569784 -> 1.84975554
Joints:
- joint j_neck_y: origin xyz=-0.004458 0.0 0.680766 rpy=0.0 0.0 0.0 -> xyz=0.00646 0.00085 0.67201 rpy=0.0 0.0 0.0

File: eve_r3_description/urdf.in/eve_r3_left_arm.in.urdf (robot description, URDF)
Before this commit: robot eve_r3_left_arm, 7 links, 7 joints
Joints:
- joint j_l_elbow_y: origin xyz=0.0 0.0 -0.313989 rpy=0.0 0.0 0.0 -> xyz=0.0 0.0 -0.3141 rpy=0.0 0.0 0.0
- joint j_l_shoulder_x: origin xyz=0.0 0.0 0.0 rpy=-0.253261563 0.0 0.0 -> xyz=0.0 0.0 0.0 rpy=-0.261799 0.0 0.0
- joint j_l_shoulder_y: origin xyz=0.010525 0.207221 0.545525 rpy=0.253261563 0.0 -0.261799 -> xyz=0.01041 0.20675 0.54735 rpy=0.261799 0.0 -0.261799

File: eve_r3_description/urdf.in/eve_r3_right_arm.in.urdf (robot description, URDF)
Before this commit: robot eve_r3_right_arm, 7 links, 7 joints
Joints:
- joint j_r_elbow_y: origin xyz=0.0 0.0 -0.313989 rpy=0.0 0.0 0.0 -> xyz=0.0 0.0 -0.3141 rpy=0.0 0.0 0.0
- joint j_r_shoulder_x: origin xyz=0.0 0.0 0.0 rpy=0.253261563 0.0 0.0 -> xyz=0.0 0.0 0.0 rpy=0.261799 0.0 0.0
- joint j_r_shoulder_y: origin xyz=0.010525 -0.207221 0.545525 rpy=-0.253261563 0.0 0.261799 -> xyz=0.01041 -0.20675 0.54735 rpy=-0.261799 0.0 0.261799
