Commit message: Converted .stl files to .obj to get URP support for free

File: eve_r3_description/urdf.in/eve_r3_head.in.urdf (robot description, URDF)
Before this commit: robot eve_r3_head, 1 links, 1 joints
Joints:
- joint j_neck_y: limit lower=-0.0872664626 upper=0.698132 effort=-1.0 velocity=-1.0 -> lower=-0.27925 upper=0.3228859 effort=-1.0 velocity=-1.0

File: eve_r3_description/urdf.in/qbhand.left.in.urdf (robot description, URDF)
Before this commit: robot qbhand_left, 36 links, 36 joints
Links:
- link qbhand_left_base_link: geometry collision mesh filename=package://qb_hand_description/meshes/flange_iso_04.obj scale=0.001 0.001 0.001; visual mesh filename=package://qb_hand_description/meshes/flange_iso_04.obj scale=0.001 0.001 0.001
- link qbhand_left_index_distal_link: geometry collision mesh filename=package://qb_hand_description/meshes/ph_distal.obj scale=0.001 0.001 0.001; visual mesh filename=package://qb_hand_description/meshes/ph_distal.obj scale=0.001 0.001 0.001
- link qbhand_left_index_knuckle_link: geometry collision mesh filename=package://qb_hand_description/meshes/ph_knuckle.obj scale=0.001 0.001 0.001; visual mesh filename=package://qb_hand_description/meshes/ph_knuckle.obj scale=0.001 0.001 0.001
- link qbhand_left_index_middle_link: geometry collision mesh filename=package://qb_hand_description/meshes/ph_small.obj scale=0.001 0.001 0.001; visual mesh filename=package://qb_hand_description/meshes/ph_small.obj scale=0.001 0.001 0.001
- link qbhand_left_index_proximal_link: geometry collision mesh filename=package://qb_hand_description/meshes/ph_medium.obj scale=0.001 0.001 0.001; visual mesh filename=package://qb_hand_description/meshes/ph_medium.obj scale=0.001 0.001 0.001
- link qbhand_left_little_distal_link: geometry collision mesh filename=package://qb_hand_description/meshes/ph_distal.obj scale=0.001 0.001 0.001; visual mesh filename=package://qb_hand_description/meshes/ph_distal.obj scale=0.001 0.001 0.001
- link qbhand_left_little_knuckle_link: geometry collision mesh filename=package://qb_hand_description/meshes/ph_knuckle.obj scale=0.001 0.001 0.001; visual mesh filename=package://qb_hand_description/meshes/ph_knuckle.obj scale=0.001 0.001 0.001
- link qbhand_left_little_middle_link: geometry collision mesh filename=package://qb_hand_description/meshes/ph_small.obj scale=0.001 0.001 0.001; visual mesh filename=package://qb_hand_description/meshes/ph_small.obj scale=0.001 0.001 0.001
- link qbhand_left_little_proximal_link: geometry collision mesh filename=package://qb_hand_description/meshes/ph_small.obj scale=0.001 0.001 0.001; visual mesh filename=package://qb_hand_description/meshes/ph_small.obj scale=0.001 0.001 0.001
- link qbhand_left_middle_distal_link: geometry collision mesh filename=package://qb_hand_description/meshes/ph_distal.obj scale=0.001 0.001 0.001; visual mesh filename=package://qb_hand_description/meshes/ph_distal.obj scale=0.001 0.001 0.001
- link qbhand_left_middle_knuckle_link: geometry collision mesh filename=package://qb_hand_description/meshes/ph_knuckle.obj scale=0.001 0.001 0.001; visual mesh filename=package://qb_hand_description/meshes/ph_knuckle.obj scale=0.001 0.001 0.001
- link qbhand_left_middle_middle_link: geometry collision mesh filename=package://qb_hand_description/meshes/ph_small.obj scale=0.001 0.001 0.001; visual mesh filename=package://qb_hand_description/meshes/ph_small.obj scale=0.001 0.001 0.001
- link qbhand_left_middle_proximal_link: geometry collision mesh filename=package://qb_hand_description/meshes/ph_medium.obj scale=0.001 0.001 0.001; visual mesh filename=package://qb_hand_description/meshes/ph_medium.obj scale=0.001 0.001 0.001
- link qbhand_left_palm_link: geometry collision mesh filename=package://qb_hand_description/meshes/palm_pinch_l.obj scale=0.001 0.001 0.001; visual mesh filename=package://qb_hand_description/meshes/palm_pinch_l.obj scale=0.001 0.001 0.001
- link qbhand_left_ring_distal_link: geometry collision mesh filename=package://qb_hand_description/meshes/ph_distal.obj scale=0.001 0.001 0.001; visual mesh filename=package://qb_hand_description/meshes/ph_distal.obj scale=0.001 0.001 0.001
- link qbhand_left_ring_knuckle_link: geometry collision mesh filename=package://qb_hand_description/meshes/ph_knuckle.obj scale=0.001 0.001 0.001; visual mesh filename=package://qb_hand_description/meshes/ph_knuckle.obj scale=0.001 0.001 0.001
- link qbhand_left_ring_middle_link: geometry collision mesh filename=package://qb_hand_description/meshes/ph_small.obj scale=0.001 0.001 0.001; visual mesh filename=package://qb_hand_description/meshes/ph_small.obj scale=0.001 0.001 0.001
- link qbhand_left_ring_proximal_link: geometry collision mesh filename=package://qb_hand_description/meshes/ph_medium.obj scale=0.001 0.001 0.001; visual mesh filename=package://qb_hand_description/meshes/ph_medium.obj scale=0.001 0.001 0.001
- link qbhand_left_thumb_distal_link: geometry collision mesh filename=package://qb_hand_description/meshes/ph_distal.obj scale=0.001 0.001 0.001; visual mesh filename=package://qb_hand_description/meshes/ph_distal.obj scale=0.001 0.001 0.001
- link qbhand_left_thumb_knuckle_link: geometry collision mesh filename=package://qb_hand_description/meshes/ph_thumb_l.obj scale=0.001 0.001 0.001; visual mesh filename=package://qb_hand_description/meshes/ph_thumb_l.obj scale=0.001 0.001 0.001
- link qbhand_left_thumb_proximal_link: geometry collision mesh filename=package://qb_hand_description/meshes/ph_small.obj scale=0.001 0.001 0.001; visual mesh filename=package://qb_hand_description/meshes/ph_small.obj scale=0.001 0.001 0.001

File: eve_r3_description/urdf.in/qbhand.right.in.urdf (robot description, URDF)
Before this commit: robot qbhand_right, 36 links, 36 joints
Links:
- link qbhand_right_base_link: geometry collision mesh filename=package://qb_hand_description/meshes/flange_iso_04.obj scale=0.001 0.001 0.001; visual mesh filename=package://qb_hand_description/meshes/flange_iso_04.obj scale=0.001 0.001 0.001
- link qbhand_right_index_distal_link: geometry collision mesh filename=package://qb_hand_description/meshes/ph_distal.obj scale=0.001 0.001 0.001; visual mesh filename=package://qb_hand_description/meshes/ph_distal.obj scale=0.001 0.001 0.001
- link qbhand_right_index_knuckle_link: geometry collision mesh filename=package://qb_hand_description/meshes/ph_knuckle.obj scale=0.001 0.001 0.001; visual mesh filename=package://qb_hand_description/meshes/ph_knuckle.obj scale=0.001 0.001 0.001
- link qbhand_right_index_middle_link: geometry collision mesh filename=package://qb_hand_description/meshes/ph_small.obj scale=0.001 0.001 0.001; visual mesh filename=package://qb_hand_description/meshes/ph_small.obj scale=0.001 0.001 0.001
- link qbhand_right_index_proximal_link: geometry collision mesh filename=package://qb_hand_description/meshes/ph_medium.obj scale=0.001 0.001 0.001; visual mesh filename=package://qb_hand_description/meshes/ph_medium.obj scale=0.001 0.001 0.001
- link qbhand_right_little_distal_link: geometry collision mesh filename=package://qb_hand_description/meshes/ph_distal.obj scale=0.001 0.001 0.001; visual mesh filename=package://qb_hand_description/meshes/ph_distal.obj scale=0.001 0.001 0.001
- link qbhand_right_little_knuckle_link: geometry collision mesh filename=package://qb_hand_description/meshes/ph_knuckle.obj scale=0.001 0.001 0.001; visual mesh filename=package://qb_hand_description/meshes/ph_knuckle.obj scale=0.001 0.001 0.001
- link qbhand_right_little_middle_link: geometry collision mesh filename=package://qb_hand_description/meshes/ph_small.obj scale=0.001 0.001 0.001; visual mesh filename=package://qb_hand_description/meshes/ph_small.obj scale=0.001 0.001 0.001
- link qbhand_right_little_proximal_link: geometry collision mesh filename=package://qb_hand_description/meshes/ph_small.obj scale=0.001 0.001 0.001; visual mesh filename=package://qb_hand_description/meshes/ph_small.obj scale=0.001 0.001 0.001
- link qbhand_right_middle_distal_link: geometry collision mesh filename=package://qb_hand_description/meshes/ph_distal.obj scale=0.001 0.001 0.001; visual mesh filename=package://qb_hand_description/meshes/ph_distal.obj scale=0.001 0.001 0.001
- link qbhand_right_middle_knuckle_link: geometry collision mesh filename=package://qb_hand_description/meshes/ph_knuckle.obj scale=0.001 0.001 0.001; visual mesh filename=package://qb_hand_description/meshes/ph_knuckle.obj scale=0.001 0.001 0.001
- link qbhand_right_middle_middle_link: geometry collision mesh filename=package://qb_hand_description/meshes/ph_small.obj scale=0.001 0.001 0.001; visual mesh filename=package://qb_hand_description/meshes/ph_small.obj scale=0.001 0.001 0.001
- link qbhand_right_middle_proximal_link: geometry collision mesh filename=package://qb_hand_description/meshes/ph_medium.obj scale=0.001 0.001 0.001; visual mesh filename=package://qb_hand_description/meshes/ph_medium.obj scale=0.001 0.001 0.001
- link qbhand_right_palm_link: geometry collision mesh filename=package://qb_hand_description/meshes/palm_pinch_r.obj scale=0.001 0.001 0.001; visual mesh filename=package://qb_hand_description/meshes/palm_pinch_r.obj scale=0.001 0.001 0.001
- link qbhand_right_ring_distal_link: geometry collision mesh filename=package://qb_hand_description/meshes/ph_distal.obj scale=0.001 0.001 0.001; visual mesh filename=package://qb_hand_description/meshes/ph_distal.obj scale=0.001 0.001 0.001
- link qbhand_right_ring_knuckle_link: geometry collision mesh filename=package://qb_hand_description/meshes/ph_knuckle.obj scale=0.001 0.001 0.001; visual mesh filename=package://qb_hand_description/meshes/ph_knuckle.obj scale=0.001 0.001 0.001
- link qbhand_right_ring_middle_link: geometry collision mesh filename=package://qb_hand_description/meshes/ph_small.obj scale=0.001 0.001 0.001; visual mesh filename=package://qb_hand_description/meshes/ph_small.obj scale=0.001 0.001 0.001
- link qbhand_right_ring_proximal_link: geometry collision mesh filename=package://qb_hand_description/meshes/ph_medium.obj scale=0.001 0.001 0.001; visual mesh filename=package://qb_hand_description/meshes/ph_medium.obj scale=0.001 0.001 0.001
- link qbhand_right_thumb_distal_link: geometry collision mesh filename=package://qb_hand_description/meshes/ph_distal.obj scale=0.001 0.001 0.001; visual mesh filename=package://qb_hand_description/meshes/ph_distal.obj scale=0.001 0.001 0.001
- link qbhand_right_thumb_knuckle_link: geometry collision mesh filename=package://qb_hand_description/meshes/ph_thumb_r.obj scale=0.001 0.001 0.001; visual mesh filename=package://qb_hand_description/meshes/ph_thumb_r.obj scale=0.001 0.001 0.001
- link qbhand_right_thumb_proximal_link: geometry collision mesh filename=package://qb_hand_description/meshes/ph_small.obj scale=0.001 0.001 0.001; visual mesh filename=package://qb_hand_description/meshes/ph_small.obj scale=0.001 0.001 0.001

File: eve_r3_description/urdf.in/robotiq_hand-e.left.in.urdf (robot description, URDF)
Before this commit: robot robotiq_hand-e, 3 links, 3 joints
Links:
- link lhand_FingerA: geometry collision box size=0.006 0.021 0.036; visual mesh filename=package://robotiq_hand-e/meshes/FingerA.obj scale=0.01 0.01 0.01
- link lhand_FingerB: geometry collision box size=0.006 0.021 0.036; visual mesh filename=package://robotiq_hand-e/meshes/FingerB.obj scale=0.01 0.01 0.01
- link lhand_base: geometry collision cylinder length=0.10005 radius=0.0375; visual mesh filename=package://robotiq_hand-e/meshes/Bolts.obj scale=0.01 0.01 0.01

File: eve_r3_description/urdf.in/robotiq_hand-e.right.in.urdf (robot description, URDF)
Before this commit: robot robotiq_hand-e, 3 links, 3 joints
Links:
- link rhand_FingerA: geometry collision box size=0.006 0.021 0.036; visual mesh filename=package://robotiq_hand-e/meshes/FingerA.obj scale=0.01 0.01 0.01
- link rhand_FingerB: geometry collision box size=0.006 0.021 0.036; visual mesh filename=package://robotiq_hand-e/meshes/FingerB.obj scale=0.01 0.01 0.01
- link rhand_base: geometry collision cylinder length=0.10005 radius=0.0375; visual mesh filename=package://robotiq_hand-e/meshes/Bolts.obj scale=0.01 0.01 0.01

File: eve_r3_description/urdf/eve_r3.urdf (robot description, URDF)
Before this commit: robot eve_r3, 96 links, 95 joints
Links:
- link qbhand_left_base_link: geometry collision mesh filename=package://qb_hand_description/meshes/flange_iso_04.obj scale=0.001 0.001 0.001; visual mesh filename=package://qb_hand_description/meshes/flange_iso_04.obj scale=0.001 0.001 0.001
- link qbhand_left_index_distal_link: geometry collision mesh filename=package://qb_hand_description/meshes/ph_distal.obj scale=0.001 0.001 0.001; visual mesh filename=package://qb_hand_description/meshes/ph_distal.obj scale=0.001 0.001 0.001
- link qbhand_left_index_knuckle_link: geometry collision mesh filename=package://qb_hand_description/meshes/ph_knuckle.obj scale=0.001 0.001 0.001; visual mesh filename=package://qb_hand_description/meshes/ph_knuckle.obj scale=0.001 0.001 0.001
- link qbhand_left_index_middle_link: geometry collision mesh filename=package://qb_hand_description/meshes/ph_small.obj scale=0.001 0.001 0.001; visual mesh filename=package://qb_hand_description/meshes/ph_small.obj scale=0.001 0.001 0.001
- link qbhand_left_index_proximal_link: geometry collision mesh filename=package://qb_hand_description/meshes/ph_medium.obj scale=0.001 0.001 0.001; visual mesh filename=package://qb_hand_description/meshes/ph_medium.obj scale=0.001 0.001 0.001
- link qbhand_left_little_distal_link: geometry collision mesh filename=package://qb_hand_description/meshes/ph_distal.obj scale=0.001 0.001 0.001; visual mesh filename=package://qb_hand_description/meshes/ph_distal.obj scale=0.001 0.001 0.001
- link qbhand_left_little_knuckle_link: geometry collision mesh filename=package://qb_hand_description/meshes/ph_knuckle.obj scale=0.001 0.001 0.001; visual mesh filename=package://qb_hand_description/meshes/ph_knuckle.obj scale=0.001 0.001 0.001
- link qbhand_left_little_middle_link: geometry collision mesh filename=package://qb_hand_description/meshes/ph_small.obj scale=0.001 0.001 0.001; visual mesh filename=package://qb_hand_description/meshes/ph_small.obj scale=0.001 0.001 0.001
- link qbhand_left_little_proximal_link: geometry collision mesh filename=package://qb_hand_description/meshes/ph_small.obj scale=0.001 0.001 0.001; visual mesh filename=package://qb_hand_description/meshes/ph_small.obj scale=0.001 0.001 0.001
- link qbhand_left_middle_distal_link: geometry collision mesh filename=package://qb_hand_description/meshes/ph_distal.obj scale=0.001 0.001 0.001; visual mesh filename=package://qb_hand_description/meshes/ph_distal.obj scale=0.001 0.001 0.001
- link qbhand_left_middle_knuckle_link: geometry collision mesh filename=package://qb_hand_description/meshes/ph_knuckle.obj scale=0.001 0.001 0.001; visual mesh filename=package://qb_hand_description/meshes/ph_knuckle.obj scale=0.001 0.001 0.001
- link qbhand_left_middle_middle_link: geometry collision mesh filename=package://qb_hand_description/meshes/ph_small.obj scale=0.001 0.001 0.001; visual mesh filename=package://qb_hand_description/meshes/ph_small.obj scale=0.001 0.001 0.001
- link qbhand_left_middle_proximal_link: geometry collision mesh filename=package://qb_hand_description/meshes/ph_medium.obj scale=0.001 0.001 0.001; visual mesh filename=package://qb_hand_description/meshes/ph_medium.obj scale=0.001 0.001 0.001
- link qbhand_left_palm_link: geometry collision mesh filename=package://qb_hand_description/meshes/palm_pinch_l.obj scale=0.001 0.001 0.001; visual mesh filename=package://qb_hand_description/meshes/palm_pinch_l.obj scale=0.001 0.001 0.001
- link qbhand_left_ring_distal_link: geometry collision mesh filename=package://qb_hand_description/meshes/ph_distal.obj scale=0.001 0.001 0.001; visual mesh filename=package://qb_hand_description/meshes/ph_distal.obj scale=0.001 0.001 0.001
- link qbhand_left_ring_knuckle_link: geometry collision mesh filename=package://qb_hand_description/meshes/ph_knuckle.obj scale=0.001 0.001 0.001; visual mesh filename=package://qb_hand_description/meshes/ph_knuckle.obj scale=0.001 0.001 0.001
- link qbhand_left_ring_middle_link: geometry collision mesh filename=package://qb_hand_description/meshes/ph_small.obj scale=0.001 0.001 0.001; visual mesh filename=package://qb_hand_description/meshes/ph_small.obj scale=0.001 0.001 0.001
- link qbhand_left_ring_proximal_link: geometry collision mesh filename=package://qb_hand_description/meshes/ph_medium.obj scale=0.001 0.001 0.001; visual mesh filename=package://qb_hand_description/meshes/ph_medium.obj scale=0.001 0.001 0.001
- link qbhand_left_thumb_distal_link: geometry collision mesh filename=package://qb_hand_description/meshes/ph_distal.obj scale=0.001 0.001 0.001; visual mesh filename=package://qb_hand_description/meshes/ph_distal.obj scale=0.001 0.001 0.001
- link qbhand_left_thumb_knuckle_link: geometry collision mesh filename=package://qb_hand_description/meshes/ph_thumb_l.obj scale=0.001 0.001 0.001; visual mesh filename=package://qb_hand_description/meshes/ph_thumb_l.obj scale=0.001 0.001 0.001
- link qbhand_left_thumb_proximal_link: geometry collision mesh filename=package://qb_hand_description/meshes/ph_small.obj scale=0.001 0.001 0.001; visual mesh filename=package://qb_hand_description/meshes/ph_small.obj scale=0.001 0.001 0.001
- link qbhand_right_base_link: geometry collision mesh filename=package://qb_hand_description/meshes/flange_iso_04.obj scale=0.001 0.001 0.001; visual mesh filename=package://qb_hand_description/meshes/flange_iso_04.obj scale=0.001 0.001 0.001
- link qbhand_right_index_distal_link: geometry collision mesh filename=package://qb_hand_description/meshes/ph_distal.obj scale=0.001 0.001 0.001; visual mesh filename=package://qb_hand_description/meshes/ph_distal.obj scale=0.001 0.001 0.001
- link qbhand_right_index_knuckle_link: geometry collision mesh filename=package://qb_hand_description/meshes/ph_knuckle.obj scale=0.001 0.001 0.001; visual mesh filename=package://qb_hand_description/meshes/ph_knuckle.obj scale=0.001 0.001 0.001
- link qbhand_right_index_middle_link: geometry collision mesh filename=package://qb_hand_description/meshes/ph_small.obj scale=0.001 0.001 0.001; visual mesh filename=package://qb_hand_description/meshes/ph_small.obj scale=0.001 0.001 0.001
- link qbhand_right_index_proximal_link: geometry collision mesh filename=package://qb_hand_description/meshes/ph_medium.obj scale=0.001 0.001 0.001; visual mesh filename=package://qb_hand_description/meshes/ph_medium.obj scale=0.001 0.001 0.001
- link qbhand_right_little_distal_link: geometry collision mesh filename=package://qb_hand_description/meshes/ph_distal.obj scale=0.001 0.001 0.001; visual mesh filename=package://qb_hand_description/meshes/ph_distal.obj scale=0.001 0.001 0.001
- link qbhand_right_little_knuckle_link: geometry collision mesh filename=package://qb_hand_description/meshes/ph_knuckle.obj scale=0.001 0.001 0.001; visual mesh filename=package://qb_hand_description/meshes/ph_knuckle.obj scale=0.001 0.001 0.001
- link qbhand_right_little_middle_link: geometry collision mesh filename=package://qb_hand_description/meshes/ph_small.obj scale=0.001 0.001 0.001; visual mesh filename=package://qb_hand_description/meshes/ph_small.obj scale=0.001 0.001 0.001
- link qbhand_right_little_proximal_link: geometry collision mesh filename=package://qb_hand_description/meshes/ph_small.obj scale=0.001 0.001 0.001; visual mesh filename=package://qb_hand_description/meshes/ph_small.obj scale=0.001 0.001 0.001
- link qbhand_right_middle_distal_link: geometry collision mesh filename=package://qb_hand_description/meshes/ph_distal.obj scale=0.001 0.001 0.001; visual mesh filename=package://qb_hand_description/meshes/ph_distal.obj scale=0.001 0.001 0.001
- link qbhand_right_middle_knuckle_link: geometry collision mesh filename=package://qb_hand_description/meshes/ph_knuckle.obj scale=0.001 0.001 0.001; visual mesh filename=package://qb_hand_description/meshes/ph_knuckle.obj scale=0.001 0.001 0.001
- link qbhand_right_middle_middle_link: geometry collision mesh filename=package://qb_hand_description/meshes/ph_small.obj scale=0.001 0.001 0.001; visual mesh filename=package://qb_hand_description/meshes/ph_small.obj scale=0.001 0.001 0.001
- link qbhand_right_middle_proximal_link: geometry collision mesh filename=package://qb_hand_description/meshes/ph_medium.obj scale=0.001 0.001 0.001; visual mesh filename=package://qb_hand_description/meshes/ph_medium.obj scale=0.001 0.001 0.001
- link qbhand_right_palm_link: geometry collision mesh filename=package://qb_hand_description/meshes/palm_pinch_r.obj scale=0.001 0.001 0.001; visual mesh filename=package://qb_hand_description/meshes/palm_pinch_r.obj scale=0.001 0.001 0.001
- link qbhand_right_ring_distal_link: geometry collision mesh filename=package://qb_hand_description/meshes/ph_distal.obj scale=0.001 0.001 0.001; visual mesh filename=package://qb_hand_description/meshes/ph_distal.obj scale=0.001 0.001 0.001
- link qbhand_right_ring_knuckle_link: geometry collision mesh filename=package://qb_hand_description/meshes/ph_knuckle.obj scale=0.001 0.001 0.001; visual mesh filename=package://qb_hand_description/meshes/ph_knuckle.obj scale=0.001 0.001 0.001
- link qbhand_right_ring_middle_link: geometry collision mesh filename=package://qb_hand_description/meshes/ph_small.obj scale=0.001 0.001 0.001; visual mesh filename=package://qb_hand_description/meshes/ph_small.obj scale=0.001 0.001 0.001
- link qbhand_right_ring_proximal_link: geometry collision mesh filename=package://qb_hand_description/meshes/ph_medium.obj scale=0.001 0.001 0.001; visual mesh filename=package://qb_hand_description/meshes/ph_medium.obj scale=0.001 0.001 0.001
- link qbhand_right_thumb_distal_link: geometry collision mesh filename=package://qb_hand_description/meshes/ph_distal.obj scale=0.001 0.001 0.001; visual mesh filename=package://qb_hand_description/meshes/ph_distal.obj scale=0.001 0.001 0.001
- link qbhand_right_thumb_knuckle_link: geometry collision mesh filename=package://qb_hand_description/meshes/ph_thumb_r.obj scale=0.001 0.001 0.001; visual mesh filename=package://qb_hand_description/meshes/ph_thumb_r.obj scale=0.001 0.001 0.001
- link qbhand_right_thumb_proximal_link: geometry collision mesh filename=package://qb_hand_description/meshes/ph_small.obj scale=0.001 0.001 0.001; visual mesh filename=package://qb_hand_description/meshes/ph_small.obj scale=0.001 0.001 0.001
Joints:
- joint j_neck_y: limit lower=-0.0872664626 upper=0.698132 effort=-1.0 velocity=-1.0 -> lower=-0.27925 upper=0.3228859 effort=-1.0 velocity=-1.0

File: eve_r3_description/urdf/eve_r3_robotiq_2f_85.urdf (robot description, URDF)
Before this commit: robot eve_r3_robotiq_2f_85, 46 links, 45 joints
Joints:
- joint j_neck_y: limit lower=-0.0872664626 upper=0.698132 effort=-1.0 velocity=-1.0 -> lower=-0.27925 upper=0.3228859 effort=-1.0 velocity=-1.0
