Commit message: Converted .stl files to .obj to get URP support for free

File: eve_r3_description/urdf/eve_r3_robotiq_hand-e.urdf (robot description, URDF)
Before this commit: robot eve_r3_robotiq_hand-e, 30 links, 29 joints
Links:
- link lhand_FingerA: geometry collision box size=0.006 0.021 0.036; visual mesh filename=package://robotiq_hand-e/meshes/FingerA.obj scale=0.01 0.01 0.01
- link lhand_FingerB: geometry collision box size=0.006 0.021 0.036; visual mesh filename=package://robotiq_hand-e/meshes/FingerB.obj scale=0.01 0.01 0.01
- link lhand_base: geometry collision cylinder length=0.10005 radius=0.0375; visual mesh filename=package://robotiq_hand-e/meshes/Bolts.obj scale=0.01 0.01 0.01
- link rhand_FingerA: geometry collision box size=0.006 0.021 0.036; visual mesh filename=package://robotiq_hand-e/meshes/FingerA.obj scale=0.01 0.01 0.01
- link rhand_FingerB: geometry collision box size=0.006 0.021 0.036; visual mesh filename=package://robotiq_hand-e/meshes/FingerB.obj scale=0.01 0.01 0.01
- link rhand_base: geometry collision cylinder length=0.10005 radius=0.0375; visual mesh filename=package://robotiq_hand-e/meshes/Bolts.obj scale=0.01 0.01 0.01
Joints:
- joint j_neck_y: limit lower=-0.0872664626 upper=0.698132 effort=-1.0 velocity=-1.0 -> lower=-0.27925 upper=0.3228859 effort=-1.0 velocity=-1.0

File: eve_r3_description/urdf/eve_r3_upper_body.urdf (robot description, URDF)
Before this commit: robot eve_r3_upper_body, 89 links, 88 joints
Links:
- link qbhand_left_base_link: geometry collision mesh filename=package://qb_hand_description/meshes/flange_iso_04.obj scale=0.001 0.001 0.001; visual mesh filename=package://qb_hand_description/meshes/flange_iso_04.obj scale=0.001 0.001 0.001
- link qbhand_left_index_distal_link: geometry collision mesh filename=package://qb_hand_description/meshes/ph_distal.obj scale=0.001 0.001 0.001; visual mesh filename=package://qb_hand_description/meshes/ph_distal.obj scale=0.001 0.001 0.001
- link qbhand_left_index_knuckle_link: geometry collision mesh filename=package://qb_hand_description/meshes/ph_knuckle.obj scale=0.001 0.001 0.001; visual mesh filename=package://qb_hand_description/meshes/ph_knuckle.obj scale=0.001 0.001 0.001
- link qbhand_left_index_middle_link: geometry collision mesh filename=package://qb_hand_description/meshes/ph_small.obj scale=0.001 0.001 0.001; visual mesh filename=package://qb_hand_description/meshes/ph_small.obj scale=0.001 0.001 0.001
- link qbhand_left_index_proximal_link: geometry collision mesh filename=package://qb_hand_description/meshes/ph_medium.obj scale=0.001 0.001 0.001; visual mesh filename=package://qb_hand_description/meshes/ph_medium.obj scale=0.001 0.001 0.001
- link qbhand_left_little_distal_link: geometry collision mesh filename=package://qb_hand_description/meshes/ph_distal.obj scale=0.001 0.001 0.001; visual mesh filename=package://qb_hand_description/meshes/ph_distal.obj scale=0.001 0.001 0.001
- link qbhand_left_little_knuckle_link: geometry collision mesh filename=package://qb_hand_description/meshes/ph_knuckle.obj scale=0.001 0.001 0.001; visual mesh filename=package://qb_hand_description/meshes/ph_knuckle.obj scale=0.001 0.001 0.001
- link qbhand_left_little_middle_link: geometry collision mesh filename=package://qb_hand_description/meshes/ph_small.obj scale=0.001 0.001 0.001; visual mesh filename=package://qb_hand_description/meshes/ph_small.obj scale=0.001 0.001 0.001
- link qbhand_left_little_proximal_link: geometry collision mesh filename=package://qb_hand_description/meshes/ph_small.obj scale=0.001 0.001 0.001; visual mesh filename=package://qb_hand_description/meshes/ph_small.obj scale=0.001 0.001 0.001
- link qbhand_left_middle_distal_link: geometry collision mesh filename=package://qb_hand_description/meshes/ph_distal.obj scale=0.001 0.001 0.001; visual mesh filename=package://qb_hand_description/meshes/ph_distal.obj scale=0.001 0.001 0.001
- link qbhand_left_middle_knuckle_link: geometry collision mesh filename=package://qb_hand_description/meshes/ph_knuckle.obj scale=0.001 0.001 0.001; visual mesh filename=package://qb_hand_description/meshes/ph_knuckle.obj scale=0.001 0.001 0.001
- link qbhand_left_middle_middle_link: geometry collision mesh filename=package://qb_hand_description/meshes/ph_small.obj scale=0.001 0.001 0.001; visual mesh filename=package://qb_hand_description/meshes/ph_small.obj scale=0.001 0.001 0.001
- link qbhand_left_middle_proximal_link: geometry collision mesh filename=package://qb_hand_description/meshes/ph_medium.obj scale=0.001 0.001 0.001; visual mesh filename=package://qb_hand_description/meshes/ph_medium.obj scale=0.001 0.001 0.001
- link qbhand_left_palm_link: geometry collision mesh filename=package://qb_hand_description/meshes/palm_pinch_l.obj scale=0.001 0.001 0.001; visual mesh filename=package://qb_hand_description/meshes/palm_pinch_l.obj scale=0.001 0.001 0.001
- link qbhand_left_ring_distal_link: geometry collision mesh filename=package://qb_hand_description/meshes/ph_distal.obj scale=0.001 0.001 0.001; visual mesh filename=package://qb_hand_description/meshes/ph_distal.obj scale=0.001 0.001 0.001
- link qbhand_left_ring_knuckle_link: geometry collision mesh filename=package://qb_hand_description/meshes/ph_knuckle.obj scale=0.001 0.001 0.001; visual mesh filename=package://qb_hand_description/meshes/ph_knuckle.obj scale=0.001 0.001 0.001
- link qbhand_left_ring_middle_link: geometry collision mesh filename=package://qb_hand_description/meshes/ph_small.obj scale=0.001 0.001 0.001; visual mesh filename=package://qb_hand_description/meshes/ph_small.obj scale=0.001 0.001 0.001
- link qbhand_left_ring_proximal_link: geometry collision mesh filename=package://qb_hand_description/meshes/ph_medium.obj scale=0.001 0.001 0.001; visual mesh filename=package://qb_hand_description/meshes/ph_medium.obj scale=0.001 0.001 0.001
- link qbhand_left_thumb_distal_link: geometry collision mesh filename=package://qb_hand_description/meshes/ph_distal.obj scale=0.001 0.001 0.001; visual mesh filename=package://qb_hand_description/meshes/ph_distal.obj scale=0.001 0.001 0.001
- link qbhand_left_thumb_knuckle_link: geometry collision mesh filename=package://qb_hand_description/meshes/ph_thumb_l.obj scale=0.001 0.001 0.001; visual mesh filename=package://qb_hand_description/meshes/ph_thumb_l.obj scale=0.001 0.001 0.001
- link qbhand_left_thumb_proximal_link: geometry collision mesh filename=package://qb_hand_description/meshes/ph_small.obj scale=0.001 0.001 0.001; visual mesh filename=package://qb_hand_description/meshes/ph_small.obj scale=0.001 0.001 0.001
- link qbhand_right_base_link: geometry collision mesh filename=package://qb_hand_description/meshes/flange_iso_04.obj scale=0.001 0.001 0.001; visual mesh filename=package://qb_hand_description/meshes/flange_iso_04.obj scale=0.001 0.001 0.001
- link qbhand_right_index_distal_link: geometry collision mesh filename=package://qb_hand_description/meshes/ph_distal.obj scale=0.001 0.001 0.001; visual mesh filename=package://qb_hand_description/meshes/ph_distal.obj scale=0.001 0.001 0.001
- link qbhand_right_index_knuckle_link: geometry collision mesh filename=package://qb_hand_description/meshes/ph_knuckle.obj scale=0.001 0.001 0.001; visual mesh filename=package://qb_hand_description/meshes/ph_knuckle.obj scale=0.001 0.001 0.001
- link qbhand_right_index_middle_link: geometry collision mesh filename=package://qb_hand_description/meshes/ph_small.obj scale=0.001 0.001 0.001; visual mesh filename=package://qb_hand_description/meshes/ph_small.obj scale=0.001 0.001 0.001
- link qbhand_right_index_proximal_link: geometry collision mesh filename=package://qb_hand_description/meshes/ph_medium.obj scale=0.001 0.001 0.001; visual mesh filename=package://qb_hand_description/meshes/ph_medium.obj scale=0.001 0.001 0.001
- link qbhand_right_little_distal_link: geometry collision mesh filename=package://qb_hand_description/meshes/ph_distal.obj scale=0.001 0.001 0.001; visual mesh filename=package://qb_hand_description/meshes/ph_distal.obj scale=0.001 0.001 0.001
- link qbhand_right_little_knuckle_link: geometry collision mesh filename=package://qb_hand_description/meshes/ph_knuckle.obj scale=0.001 0.001 0.001; visual mesh filename=package://qb_hand_description/meshes/ph_knuckle.obj scale=0.001 0.001 0.001
- link qbhand_right_little_middle_link: geometry collision mesh filename=package://qb_hand_description/meshes/ph_small.obj scale=0.001 0.001 0.001; visual mesh filename=package://qb_hand_description/meshes/ph_small.obj scale=0.001 0.001 0.001
- link qbhand_right_little_proximal_link: geometry collision mesh filename=package://qb_hand_description/meshes/ph_small.obj scale=0.001 0.001 0.001; visual mesh filename=package://qb_hand_description/meshes/ph_small.obj scale=0.001 0.001 0.001
- link qbhand_right_middle_distal_link: geometry collision mesh filename=package://qb_hand_description/meshes/ph_distal.obj scale=0.001 0.001 0.001; visual mesh filename=package://qb_hand_description/meshes/ph_distal.obj scale=0.001 0.001 0.001
- link qbhand_right_middle_knuckle_link: geometry collision mesh filename=package://qb_hand_description/meshes/ph_knuckle.obj scale=0.001 0.001 0.001; visual mesh filename=package://qb_hand_description/meshes/ph_knuckle.obj scale=0.001 0.001 0.001
- link qbhand_right_middle_middle_link: geometry collision mesh filename=package://qb_hand_description/meshes/ph_small.obj scale=0.001 0.001 0.001; visual mesh filename=package://qb_hand_description/meshes/ph_small.obj scale=0.001 0.001 0.001
- link qbhand_right_middle_proximal_link: geometry collision mesh filename=package://qb_hand_description/meshes/ph_medium.obj scale=0.001 0.001 0.001; visual mesh filename=package://qb_hand_description/meshes/ph_medium.obj scale=0.001 0.001 0.001
- link qbhand_right_palm_link: geometry collision mesh filename=package://qb_hand_description/meshes/palm_pinch_r.obj scale=0.001 0.001 0.001; visual mesh filename=package://qb_hand_description/meshes/palm_pinch_r.obj scale=0.001 0.001 0.001
- link qbhand_right_ring_distal_link: geometry collision mesh filename=package://qb_hand_description/meshes/ph_distal.obj scale=0.001 0.001 0.001; visual mesh filename=package://qb_hand_description/meshes/ph_distal.obj scale=0.001 0.001 0.001
- link qbhand_right_ring_knuckle_link: geometry collision mesh filename=package://qb_hand_description/meshes/ph_knuckle.obj scale=0.001 0.001 0.001; visual mesh filename=package://qb_hand_description/meshes/ph_knuckle.obj scale=0.001 0.001 0.001
- link qbhand_right_ring_middle_link: geometry collision mesh filename=package://qb_hand_description/meshes/ph_small.obj scale=0.001 0.001 0.001; visual mesh filename=package://qb_hand_description/meshes/ph_small.obj scale=0.001 0.001 0.001
- link qbhand_right_ring_proximal_link: geometry collision mesh filename=package://qb_hand_description/meshes/ph_medium.obj scale=0.001 0.001 0.001; visual mesh filename=package://qb_hand_description/meshes/ph_medium.obj scale=0.001 0.001 0.001
- link qbhand_right_thumb_distal_link: geometry collision mesh filename=package://qb_hand_description/meshes/ph_distal.obj scale=0.001 0.001 0.001; visual mesh filename=package://qb_hand_description/meshes/ph_distal.obj scale=0.001 0.001 0.001
- link qbhand_right_thumb_knuckle_link: geometry collision mesh filename=package://qb_hand_description/meshes/ph_thumb_r.obj scale=0.001 0.001 0.001; visual mesh filename=package://qb_hand_description/meshes/ph_thumb_r.obj scale=0.001 0.001 0.001
- link qbhand_right_thumb_proximal_link: geometry collision mesh filename=package://qb_hand_description/meshes/ph_small.obj scale=0.001 0.001 0.001; visual mesh filename=package://qb_hand_description/meshes/ph_small.obj scale=0.001 0.001 0.001
Joints:
- joint j_neck_y: limit lower=-0.0872664626 upper=0.698132 effort=-1.0 velocity=-1.0 -> lower=-0.27925 upper=0.3228859 effort=-1.0 velocity=-1.0

File: halodi-robot-models-unity-support/Packages/halodi-robot-models/Runtime/Halodi/Models/robotiq_hand-e.urdf (robot description, URDF)
Before this commit: robot robotiq_hand-e, 3 links, 2 joints
Links:
- link FingerA: geometry collision box size=0.006 0.021 0.036; visual mesh filename=package://robotiq_hand-e/meshes/FingerA.obj scale=0.01 0.01 0.01
- link FingerB: geometry collision box size=0.006 0.021 0.036; visual mesh filename=package://robotiq_hand-e/meshes/FingerB.obj scale=0.01 0.01 0.01
- link base: geometry collision cylinder length=0.10005 radius=0.0375; visual mesh filename=package://robotiq_hand-e/meshes/Bolts.obj scale=0.01 0.01 0.01

File: robotiq_2f_85_gripper_visualization/urdf/robotiq_arg2f.xacro (robot description, xacro)
@@ -20,5 +20,5 @@
         <origin xyz="0 0 0" rpy="0 0 0" />
         <geometry>
-           <mesh filename="package://robotiq_2f_85_gripper_visualization/meshes/collision/robotiq_arg2f_base_link.stl" />
+           <mesh filename="package://robotiq_2f_85_gripper_visualization/meshes/collision/robotiq_arg2f_base_link.obj" />
         </geometry>
       </collision>

Commit message: Updated neck limits

File: eve_r3_description/urdf.in/eve_r3_head.in.urdf (robot description, URDF)
Before this commit: robot eve_r3_head, 1 links, 1 joints
Joints:
- joint j_neck_y: limit lower=-0.27925 upper=0.3228859 effort=-1.0 velocity=-1.0 -> lower=-0.335 upper=0.506 effort=-1.0 velocity=-1.0

File: eve_r3_description/urdf/eve_r3.urdf (robot description, URDF)
Before this commit: robot eve_r3, 96 links, 95 joints
Joints:
- joint j_neck_y: limit lower=-0.27925 upper=0.3228859 effort=-1.0 velocity=-1.0 -> lower=-0.335 upper=0.506 effort=-1.0 velocity=-1.0

File: eve_r3_description/urdf/eve_r3_robotiq_2f_85.urdf (robot description, URDF)
Before this commit: robot eve_r3_robotiq_2f_85, 46 links, 45 joints
Joints:
- joint j_neck_y: limit lower=-0.27925 upper=0.3228859 effort=-1.0 velocity=-1.0 -> lower=-0.335 upper=0.506 effort=-1.0 velocity=-1.0

File: eve_r3_description/urdf/eve_r3_robotiq_hand-e.urdf (robot description, URDF)
Before this commit: robot eve_r3_robotiq_hand-e, 30 links, 29 joints
Joints:
- joint j_neck_y: limit lower=-0.27925 upper=0.3228859 effort=-1.0 velocity=-1.0 -> lower=-0.335 upper=0.506 effort=-1.0 velocity=-1.0

File: eve_r3_description/urdf/eve_r3_upper_body.urdf (robot description, URDF)
Before this commit: robot eve_r3_upper_body, 89 links, 88 joints
Joints:
- joint j_neck_y: limit lower=-0.27925 upper=0.3228859 effort=-1.0 velocity=-1.0 -> lower=-0.335 upper=0.506 effort=-1.0 velocity=-1.0

Commit message: Updated neck angle limits to match CAD

File: eve_r3_description/urdf.in/eve_r3_head.in.urdf (robot description, URDF)
Before this commit: robot eve_r3_head, 1 links, 1 joints
Joints:
- joint j_neck_y: limit lower=-0.335 upper=0.506 effort=-1.0 velocity=-1.0 -> lower=-0.3054 upper=0.480 effort=-1.0 velocity=-1.0

File: eve_r3_description/urdf/eve_r3.urdf (robot description, URDF)
Before this commit: robot eve_r3, 96 links, 95 joints
Joints:
- joint j_neck_y: limit lower=-0.335 upper=0.506 effort=-1.0 velocity=-1.0 -> lower=-0.3054 upper=0.480 effort=-1.0 velocity=-1.0

File: eve_r3_description/urdf/eve_r3_robotiq_2f_85.urdf (robot description, URDF)
Before this commit: robot eve_r3_robotiq_2f_85, 46 links, 45 joints
Joints:
- joint j_neck_y: limit lower=-0.335 upper=0.506 effort=-1.0 velocity=-1.0 -> lower=-0.3054 upper=0.480 effort=-1.0 velocity=-1.0

File: eve_r3_description/urdf/eve_r3_robotiq_hand-e.urdf (robot description, URDF)
Before this commit: robot eve_r3_robotiq_hand-e, 30 links, 29 joints
Joints:
- joint j_neck_y: limit lower=-0.335 upper=0.506 effort=-1.0 velocity=-1.0 -> lower=-0.3054 upper=0.480 effort=-1.0 velocity=-1.0

File: eve_r3_description/urdf/eve_r3_upper_body.urdf (robot description, URDF)
Before this commit: robot eve_r3_upper_body, 89 links, 88 joints
Joints:
- joint j_neck_y: limit lower=-0.335 upper=0.506 effort=-1.0 velocity=-1.0 -> lower=-0.3054 upper=0.480 effort=-1.0 velocity=-1.0

Commit message: Revert "Updated neck angle limits to match CAD"
This reverts commit e9c6c98c678151fc674eea90de1aea3e9939e298.

File: eve_r3_description/urdf.in/eve_r3_head.in.urdf (robot description, URDF)
Before this commit: robot eve_r3_head, 1 links, 1 joints
Joints:
- joint j_neck_y: limit lower=-0.3054 upper=0.480 effort=-1.0 velocity=-1.0 -> lower=-0.335 upper=0.506 effort=-1.0 velocity=-1.0

File: eve_r3_description/urdf/eve_r3.urdf (robot description, URDF)
Before this commit: robot eve_r3, 96 links, 95 joints
Joints:
- joint j_neck_y: limit lower=-0.3054 upper=0.480 effort=-1.0 velocity=-1.0 -> lower=-0.335 upper=0.506 effort=-1.0 velocity=-1.0

File: eve_r3_description/urdf/eve_r3_robotiq_2f_85.urdf (robot description, URDF)
Before this commit: robot eve_r3_robotiq_2f_85, 46 links, 45 joints
Joints:
- joint j_neck_y: limit lower=-0.3054 upper=0.480 effort=-1.0 velocity=-1.0 -> lower=-0.335 upper=0.506 effort=-1.0 velocity=-1.0

File: eve_r3_description/urdf/eve_r3_robotiq_hand-e.urdf (robot description, URDF)
Before this commit: robot eve_r3_robotiq_hand-e, 30 links, 29 joints
Joints:
- joint j_neck_y: limit lower=-0.3054 upper=0.480 effort=-1.0 velocity=-1.0 -> lower=-0.335 upper=0.506 effort=-1.0 velocity=-1.0

File: eve_r3_description/urdf/eve_r3_upper_body.urdf (robot description, URDF)
Before this commit: robot eve_r3_upper_body, 89 links, 88 joints
Joints:
- joint j_neck_y: limit lower=-0.3054 upper=0.480 effort=-1.0 velocity=-1.0 -> lower=-0.335 upper=0.506 effort=-1.0 velocity=-1.0
