Commit message: Added hand-e hand from robotiq

File: eve_r3_description/urdf.in/robotiq_2f_85.left.in.urdf (robot description, URDF)
Before this commit: robot robotiq_arg2f_85_model, 11 links, 11 joints
Joints:
- joint lhand_robotiq_2f_85_right_base_fixed_joint: origin xyz=0 0 0 rpy=0 0 0 -> xyz=0 0 -0.06 rpy=3.14 0 0

File: eve_r3_description/urdf.in/robotiq_2f_85.right.in.urdf (robot description, URDF)
Before this commit: robot robotiq_arg2f_85_model, 11 links, 11 joints
Joints:
- joint rhand_robotiq_2f_85_right_base_fixed_joint: origin xyz=0 0 0 rpy=0 0 0 -> xyz=0 0 -0.06 rpy=3.14 0 0

Commit message: Implemented support for articulation bodies for a stable simulation.
Removed ROS# elements from exported models and replaced with custom ArticulationJoint to allow switching between dynamic/kinematic mode. Added Robotiq hands for manipulation testing.

File: eve_r3_description/urdf.in/robotiq_2f_85.left.in.urdf (robot description, URDF)
Before this commit: robot robotiq_arg2f_85_model, 11 links, 11 joints
Links:
- link lhand_left_inner_finger: mass None -> 0.0104003125914103; geometry visual mesh filename=package://robotiq_2f_85_gripper_visualization/meshes/visual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 scale=0.001 0.001 0.001
- link lhand_left_inner_knuckle: mass None -> 0.0271177346495152
- link lhand_left_outer_finger: mass None -> 0.022614240507152
- link lhand_left_outer_knuckle: mass None -> 0.00853198276973456; geometry visual mesh filename=package://robotiq_2f_85_gripper_visualization/meshes/visual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 scale=0.001 0.001 0.001
- link lhand_right_inner_finger: mass None -> 0.0104003125914103; geometry visual mesh filename=package://robotiq_2f_85_gripper_visualization/meshes/visual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 scale=0.001 0.001 0.001
- link lhand_right_inner_knuckle: mass None -> 0.0271177346495152
- link lhand_right_outer_finger: mass None -> 0.022614240507152
- link lhand_right_outer_knuckle: mass None -> 0.00853198276973456; geometry visual mesh filename=package://robotiq_2f_85_gripper_visualization/meshes/visual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 scale=0.001 0.001 0.001
Joints:
- joint lhand_left_inner_finger_joint: type revolute -> continuous
- joint lhand_left_outer_finger_joint: limit (none) -> lower=-3.14 upper=0 effort=1000 velocity=2.0; type fixed -> revolute
- joint lhand_right_inner_finger_joint: type revolute -> continuous
- joint lhand_right_outer_finger_joint: limit (none) -> lower=-3.14 upper=0 effort=1000 velocity=2.0; type fixed -> revolute

File: eve_r3_description/urdf.in/robotiq_2f_85.right.in.urdf (robot description, URDF)
Before this commit: robot robotiq_arg2f_85_model, 11 links, 11 joints
Links:
- link rhand_left_inner_finger: mass None -> 0.0104003125914103; geometry visual mesh filename=package://robotiq_2f_85_gripper_visualization/meshes/visual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 scale=0.001 0.001 0.001
- link rhand_left_inner_knuckle: mass None -> 0.0271177346495152
- link rhand_left_outer_finger: mass None -> 0.022614240507152
- link rhand_left_outer_knuckle: mass None -> 0.00853198276973456; geometry visual mesh filename=package://robotiq_2f_85_gripper_visualization/meshes/visual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 scale=0.001 0.001 0.001
- link rhand_right_inner_finger: mass None -> 0.0104003125914103; geometry visual mesh filename=package://robotiq_2f_85_gripper_visualization/meshes/visual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 scale=0.001 0.001 0.001
- link rhand_right_inner_knuckle: mass None -> 0.0271177346495152
- link rhand_right_outer_finger: mass None -> 0.022614240507152
- link rhand_right_outer_knuckle: mass None -> 0.00853198276973456; geometry visual mesh filename=package://robotiq_2f_85_gripper_visualization/meshes/visual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 scale=0.001 0.001 0.001
Joints:
- joint rhand_left_inner_finger_joint: type revolute -> continuous
- joint rhand_left_outer_finger_joint: limit (none) -> lower=-3.14 upper=0 effort=1000 velocity=2.0; type fixed -> revolute
- joint rhand_right_inner_finger_joint: type revolute -> continuous
- joint rhand_right_outer_finger_joint: limit (none) -> lower=-3.14 upper=0 effort=1000 velocity=2.0; type fixed -> revolute

File: eve_r3_description/urdf.in/robotiq_hand-e.left.in.urdf (robot description, URDF)
Before this commit: robot robotiq_hand-e, 3 links, 3 joints
Joints:
- joint lhand_fingerA_joint: axis 0 -1 0 -> -1 0 0
- joint lhand_fingerB_joint: axis 0 -1 0 -> 1 0 0; limit lower=-0.025 upper=0.0 effort=1000 velocity=1000 -> lower=0.0 upper=0.025 effort=1000 velocity=1000

File: eve_r3_description/urdf.in/robotiq_hand-e.right.in.urdf (robot description, URDF)
Before this commit: robot robotiq_hand-e, 3 links, 3 joints
Joints:
- joint rhand_fingerA_joint: axis 0 -1 0 -> -1 0 0
- joint rhand_fingerB_joint: axis 0 -1 0 -> 1 0 0; limit lower=-0.025 upper=0.0 effort=1000 velocity=1000 -> lower=0.0 upper=0.025 effort=1000 velocity=1000

Commit message: set robotiq joints to fixed

File: eve_r3_description/urdf.in/robotiq_2f_85.left.in.urdf (robot description, URDF)
Before this commit: robot robotiq_arg2f_85_model, 11 links, 11 joints
Joints:
- joint lhand_finger_joint: type revolute -> fixed
- joint lhand_left_inner_knuckle_joint: type revolute -> fixed
- joint lhand_left_outer_finger_joint: type revolute -> fixed
- joint lhand_right_inner_knuckle_joint: type revolute -> fixed
- joint lhand_right_outer_finger_joint: type revolute -> fixed
- joint lhand_right_outer_knuckle_joint: type revolute -> fixed

File: eve_r3_description/urdf.in/robotiq_2f_85.right.in.urdf (robot description, URDF)
Before this commit: robot robotiq_arg2f_85_model, 11 links, 11 joints
Joints:
- joint rhand_finger_joint: type revolute -> fixed
- joint rhand_left_inner_knuckle_joint: type revolute -> fixed
- joint rhand_left_outer_finger_joint: type revolute -> fixed
- joint rhand_right_inner_knuckle_joint: type revolute -> fixed
- joint rhand_right_outer_finger_joint: type revolute -> fixed
- joint rhand_right_outer_knuckle_joint: type revolute -> fixed

File: eve_r3_description/urdf.in/robotiq_hand-e.left.in.urdf (robot description, URDF)
Before this commit: robot robotiq_hand-e, 3 links, 3 joints
Joints:
- joint lhand_fingerA_joint: type prismatic -> fixed
- joint lhand_fingerB_joint: type prismatic -> fixed

File: eve_r3_description/urdf.in/robotiq_hand-e.right.in.urdf (robot description, URDF)
Before this commit: robot robotiq_hand-e, 3 links, 3 joints
Joints:
- joint rhand_fingerA_joint: type prismatic -> fixed
- joint rhand_fingerB_joint: type prismatic -> fixed

File: eve_r3_description/urdf/eve_r3_robotiq_2f_85.urdf (robot description, URDF)
Before this commit: robot eve_r3_robotiq_2f_85, 46 links, 45 joints
Joints:
- joint lhand_finger_joint: type revolute -> fixed
- joint lhand_left_inner_knuckle_joint: type revolute -> fixed
- joint lhand_left_outer_finger_joint: type revolute -> fixed
- joint lhand_right_inner_knuckle_joint: type revolute -> fixed
- joint lhand_right_outer_finger_joint: type revolute -> fixed
- joint lhand_right_outer_knuckle_joint: type revolute -> fixed
- joint rhand_finger_joint: type revolute -> fixed
- joint rhand_left_inner_knuckle_joint: type revolute -> fixed
- joint rhand_left_outer_finger_joint: type revolute -> fixed
- joint rhand_right_inner_knuckle_joint: type revolute -> fixed
- joint rhand_right_outer_finger_joint: type revolute -> fixed
- joint rhand_right_outer_knuckle_joint: type revolute -> fixed

File: eve_r3_description/urdf/eve_r3_robotiq_hand-e.urdf (robot description, URDF)
Before this commit: robot eve_r3_robotiq_hand-e, 30 links, 29 joints
Joints:
- joint lhand_fingerA_joint: type prismatic -> fixed
- joint lhand_fingerB_joint: type prismatic -> fixed
- joint rhand_fingerA_joint: type prismatic -> fixed
- joint rhand_fingerB_joint: type prismatic -> fixed

Commit message: fill all robotiq joints

File: eve_r3_description/urdf.in/robotiq_2f_85.left.in.urdf (robot description, URDF)
Before this commit: robot robotiq_arg2f_85_model, 11 links, 11 joints
Joints:
- joint lhand_left_inner_finger_joint: type continuous -> fixed
- joint lhand_right_inner_finger_joint: type continuous -> fixed

File: eve_r3_description/urdf.in/robotiq_2f_85.right.in.urdf (robot description, URDF)
Before this commit: robot robotiq_arg2f_85_model, 11 links, 11 joints
Joints:
- joint rhand_left_inner_finger_joint: type continuous -> fixed
- joint rhand_right_inner_finger_joint: type continuous -> fixed

Commit message: make all joints fixed

File: eve_r3_description/urdf.in/robotiq_2f_85.left.in.urdf (robot description, URDF)
Before this commit: robot robotiq_arg2f_85_model, 11 links, 11 joints
Joints:
- joint lhand_finger_joint: type revolute -> fixed
- joint lhand_left_inner_finger_joint: type continuous -> fixed
- joint lhand_left_inner_knuckle_joint: type revolute -> fixed
- joint lhand_left_outer_finger_joint: type revolute -> fixed
- joint lhand_right_inner_finger_joint: type continuous -> fixed
- joint lhand_right_inner_knuckle_joint: type revolute -> fixed
- joint lhand_right_outer_finger_joint: type revolute -> fixed
- joint lhand_right_outer_knuckle_joint: type revolute -> fixed

File: eve_r3_description/urdf.in/robotiq_2f_85.right.in.urdf (robot description, URDF)
Before this commit: robot robotiq_arg2f_85_model, 11 links, 11 joints
Joints:
- joint rhand_finger_joint: type revolute -> fixed
- joint rhand_left_inner_finger_joint: type continuous -> fixed
- joint rhand_left_inner_knuckle_joint: type revolute -> fixed
- joint rhand_left_outer_finger_joint: type revolute -> fixed
- joint rhand_right_inner_finger_joint: type continuous -> fixed
- joint rhand_right_inner_knuckle_joint: type revolute -> fixed
- joint rhand_right_outer_finger_joint: type revolute -> fixed
- joint rhand_right_outer_knuckle_joint: type revolute -> fixed

File: robotiq_2f_85_gripper_visualization/urdf/robotiq_arg2f_85_model_macro.xacro (robot description, xacro)
@@ -130,5 +130,5 @@
   </xacro:macro>
   <xacro:macro name="inner_knuckle_joint" params="prefix fingerprefix reflect">
-    <joint name="${prefix}${fingerprefix}_inner_knuckle_joint" type="revolute">
+    <joint name="${prefix}${fingerprefix}_inner_knuckle_joint" type="fixed">
       <!-- <origin xyz="0 ${reflect * -0.0127} 0.06142" rpy="${pi / 2 + .725} 0 ${(reflect - 1) * pi / 2}" /> -->
       <origin xyz="0 ${reflect * -0.0127} 0.06142" rpy="0 0 ${(1 + reflect) * pi / 2}"/>
@@ -141,5 +141,5 @@
   </xacro:macro>
   <xacro:macro name="inner_finger_joint" params="prefix fingerprefix">
-    <joint name="${prefix}${fingerprefix}_inner_finger_joint" type="revolute">
+    <joint name="${prefix}${fingerprefix}_inner_finger_joint" type="fixed">
       <origin xyz="0 0.0061 0.0471" rpy="0 0 0"/>
       <parent link="${prefix}${fingerprefix}_outer_finger" />
@@ -160,5 +160,5 @@
   <xacro:include filename="$(find robotiq_2f_85_gripper_visualization)/urdf/robotiq_arg2f.xacro" />
   <xacro:macro name="finger_joint" params="prefix">
-    <joint name="${prefix}finger_joint" type="revolute">
+    <joint name="${prefix}finger_joint" type="fixed">
       <origin xyz="0 -0.0306011 0.054904" rpy="0 0 ${pi}"/>
       <parent link="${prefix}robotiq_arg2f_base_link" />
@@ -170,5 +170,5 @@
   </xacro:macro>
   <xacro:macro name="right_outer_knuckle_joint" params="prefix">
-    <joint name="${prefix}right_outer_knuckle_joint" type="revolute">
+    <joint name="${prefix}right_outer_knuckle_joint" type="fixed">
       <origin xyz="0 0.0306011 0.054904" rpy="0 0 0"/>
       <parent link="${prefix}robotiq_arg2f_base_link" />
