Commit message: Adjust caster collision sphere

File: eve_r3_description/urdf.in/eve_r3_leg.collision.in.urdf (robot description, URDF)
Before this commit: robot eve_r3_leg, 9 links, 8 joints
Links:
- link base: geometry collision sphere radius=0.1; visual mesh filename=package://eve_r3_description/meshes/base.obj scale=1 1 1

File: eve_r3_description/urdf/eve_r3.collision.urdf (robot description, URDF)
Before this commit: robot eve_r3, 96 links, 95 joints
Links:
- link base: geometry collision sphere radius=0.1; visual mesh filename=package://eve_r3_description/meshes/base.obj scale=1 1 1

File: eve_r3_description/urdf/xacro/eve_r3.collision.urdf.xacro (robot description, xacro)
@@ -170,7 +170,7 @@
     </visual>
     <collision>
-      <origin xyz="-0.284 0.0 0.019000" rpy="0.0 0.0 0.0"/>
-      <geometry>
-        <sphere radius="0.1524"/>
+      <origin xyz="-0.284 0.0 -0.0334" rpy="0.0 0.0 0.0"/>
+      <geometry>
+        <sphere radius="0.1"/>
       </geometry>
     </collision>
