Commit message: Updated eve2019 robot model with upper body models. Default render pipeline

File: halodi-robot-models-unity-support/Assets/halodi-robot-models/Runtime/halodi/models/eve_r3_upper_body.urdf (robot description, URDF)
Before this commit: robot eve_r3_upper_body, 87 links, 86 joints
Links:
- added link abdomen, mass 3.4381772; visual mesh filename=package://eve_r3_description/meshes/abdomen.obj scale=1 1 1
- added link head, mass 2.355; visual mesh filename=package://eve_r3_description/meshes/head.obj scale=1 1 1
Joints:
- added joint j_hip_z: type revolute, parent abdomen, child pelvis, origin xyz=0.0 0.0 0.0 rpy=0.0 0.0 0.0, axis 0.0 0.0 1.0, limit lower=-1.0472 upper=1.0472 effort=-1.0 velocity=-1.0
- added joint j_neck_y: type revolute, parent pelvis, child head, origin xyz=-0.004458 0.0 0.680766 rpy=0.0 0.0 0.0, axis 0.0 1 0.0, limit lower=-0.0872664626 upper=0.698132 effort=-1.0 velocity=-1.0
