Commit message: regenerate sdf

File: eve_r3_description/urdf/eve_r3_robotiq_2f_85.urdf (robot description, URDF)
Before this commit: robot eve_r3_robotiq_2f_85, 46 links, 45 joints
Joints:
- joint lhand_finger_joint: type revolute -> fixed
- joint lhand_left_inner_finger_joint: type continuous -> fixed
- joint lhand_left_inner_knuckle_joint: type revolute -> fixed
- joint lhand_left_outer_finger_joint: type revolute -> fixed
- joint lhand_right_inner_finger_joint: type continuous -> fixed
- joint lhand_right_inner_knuckle_joint: type revolute -> fixed
- joint lhand_right_outer_finger_joint: type revolute -> fixed
- joint lhand_right_outer_knuckle_joint: type revolute -> fixed
- joint rhand_finger_joint: type revolute -> fixed
- joint rhand_left_inner_finger_joint: type continuous -> fixed
- joint rhand_left_inner_knuckle_joint: type revolute -> fixed
- joint rhand_left_outer_finger_joint: type revolute -> fixed
- joint rhand_right_inner_finger_joint: type continuous -> fixed
- joint rhand_right_inner_knuckle_joint: type revolute -> fixed
- joint rhand_right_outer_finger_joint: type revolute -> fixed
- joint rhand_right_outer_knuckle_joint: type revolute -> fixed

Commit message: update robotiq dae paths in urdf

File: eve_r3_description/urdf/eve_r3_robotiq_2f_85.urdf (robot description, URDF)
Before this commit: robot eve_r3_robotiq_2f_85, 46 links, 45 joints
Links:
- link lhand_left_inner_finger: geometry visual mesh filename=package://robotiq_2f_85_gripper_visualization/models/roboti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 scale=0.001 0.001 0.001
- link lhand_left_inner_knuckle: geometry collision mesh filename=package://robotiq_2f_85_gripper_visualization/models/roboti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 scale=0.001 0.001 0.001; visual mesh filename=package://robotiq_2f_85_gripper_visualization/models/roboti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 scale=0.001 0.001 0.001
- link lhand_left_outer_finger: geometry collision mesh filename=package://robotiq_2f_85_gripper_visualization/models/roboti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 scale=0.001 0.001 0.001; visual mesh filename=package://robotiq_2f_85_gripper_visualization/models/roboti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 scale=0.001 0.001 0.001
- link lhand_left_outer_knuckle: geometry visual mesh filename=package://robotiq_2f_85_gripper_visualization/models/roboti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 scale=0.001 0.001 0.001
- link lhand_right_inner_finger: geometry visual mesh filename=package://robotiq_2f_85_gripper_visualization/models/roboti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 scale=0.001 0.001 0.001
- link lhand_right_inner_knuckle: geometry collision mesh filename=package://robotiq_2f_85_gripper_visualization/models/roboti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 scale=0.001 0.001 0.001; visual mesh filename=package://robotiq_2f_85_gripper_visualization/models/roboti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 scale=0.001 0.001 0.001
- link lhand_right_outer_finger: geometry collision mesh filename=package://robotiq_2f_85_gripper_visualization/models/roboti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 scale=0.001 0.001 0.001; visual mesh filename=package://robotiq_2f_85_gripper_visualization/models/roboti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 scale=0.001 0.001 0.001
- link lhand_right_outer_knuckle: geometry visual mesh filename=package://robotiq_2f_85_gripper_visualization/models/roboti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 scale=0.001 0.001 0.001
- link lhand_robotiq_arg2f_base_link: geometry collision mesh filename=package://robotiq_2f_85_gripper_visualization/models/roboti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; visual mesh filename=package://robotiq_2f_85_gripper_visualization/models/roboti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 scale=0.001 0.001 0.001
- link rhand_left_inner_finger: geometry visual mesh filename=package://robotiq_2f_85_gripper_visualization/models/roboti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 scale=0.001 0.001 0.001
- link rhand_left_inner_knuckle: geometry collision mesh filename=package://robotiq_2f_85_gripper_visualization/models/roboti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 scale=0.001 0.001 0.001; visual mesh filename=package://robotiq_2f_85_gripper_visualization/models/roboti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 scale=0.001 0.001 0.001
- link rhand_left_outer_finger: geometry collision mesh filename=package://robotiq_2f_85_gripper_visualization/models/roboti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 scale=0.001 0.001 0.001; visual mesh filename=package://robotiq_2f_85_gripper_visualization/models/roboti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 scale=0.001 0.001 0.001
- link rhand_left_outer_knuckle: geometry visual mesh filename=package://robotiq_2f_85_gripper_visualization/models/roboti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 scale=0.001 0.001 0.001
- link rhand_right_inner_finger: geometry visual mesh filename=package://robotiq_2f_85_gripper_visualization/models/roboti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 scale=0.001 0.001 0.001
- link rhand_right_inner_knuckle: geometry collision mesh filename=package://robotiq_2f_85_gripper_visualization/models/roboti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 scale=0.001 0.001 0.001; visual mesh filename=package://robotiq_2f_85_gripper_visualization/models/roboti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 scale=0.001 0.001 0.001
- link rhand_right_outer_finger: geometry collision mesh filename=package://robotiq_2f_85_gripper_visualization/models/roboti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 scale=0.001 0.001 0.001; visual mesh filename=package://robotiq_2f_85_gripper_visualization/models/roboti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 scale=0.001 0.001 0.001
- link rhand_right_outer_knuckle: geometry visual mesh filename=package://robotiq_2f_85_gripper_visualization/models/roboti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 scale=0.001 0.001 0.001
- link rhand_robotiq_arg2f_base_link: geometry collision mesh filename=package://robotiq_2f_85_gripper_visualization/models/roboti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; visual mesh filename=package://robotiq_2f_85_gripper_visualization/models/roboti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 scale=0.001 0.001 0.001

Commit message: Set robotiq revolute joints to fixed

File: eve_r3_description/urdf/eve_r3_robotiq_2f_85.urdf (robot description, URDF)
Before this commit: robot eve_r3_robotiq_2f_85, 46 links, 45 joints
Joints:
- joint lhand_finger_joint: type revolute -> fixed
- joint lhand_left_inner_knuckle_joint: type revolute -> fixed
- joint lhand_left_outer_finger_joint: type revolute -> fixed
- joint lhand_right_inner_knuckle_joint: type revolute -> fixed
- joint lhand_right_outer_finger_joint: type revolute -> fixed
- joint lhand_right_outer_knuckle_joint: type revolute -> fixed
- joint rhand_finger_joint: type revolute -> fixed
- joint rhand_left_inner_knuckle_joint: type revolute -> fixed
- joint rhand_left_outer_finger_joint: type revolute -> fixed
- joint rhand_right_inner_knuckle_joint: type revolute -> fixed
- joint rhand_right_outer_finger_joint: type revolute -> fixed
- joint rhand_right_outer_knuckle_joint: type revolute -> fixed

Commit message: Set robotiq continuous joints to fixed

File: eve_r3_description/urdf/eve_r3_robotiq_2f_85.urdf (robot description, URDF)
Before this commit: robot eve_r3_robotiq_2f_85, 46 links, 45 joints
Joints:
- joint lhand_left_inner_finger_joint: type continuous -> fixed
- joint lhand_right_inner_finger_joint: type continuous -> fixed
- joint rhand_left_inner_finger_joint: type continuous -> fixed
- joint rhand_right_inner_finger_joint: type continuous -> fixed
